Commit message: labor 26./27.08.: erfolgsraten-logging, timeout_is_failure, tastatur-fallback
- Lernkurve als Erfolgsrate statt ep_rew_mean: is_success im Env,
  SuccessRateCallback, VecMonitor(info_keywords), eval/plot_success_curve.py.
  ep_rew_mean ist bimodal und taugt nicht als Fortschrittsanzeige.
- timeout_is_failure in beiden *_neutraining.yaml: Timeout ohne bestaetigten
  Trigger zaehlt als Fehlschlag, damit der Griffabschluss ueberhaupt einen
  Gradienten bekommt. Precision lernt das erst ab ~1.25M Steps, davor 0 %.
  Die *_realmatch.yaml messen dagegen mit dem Massstab von policy_runner.py,
  der real auch ohne Trigger anhebt.
- ppo_final.yaml (eval_freq 25k) und ppo_finegrain.yaml (200k, eval_freq 5k):
  eval_freq 100k legt den ganzen Lernvorgang ins erste Messintervall.
  Beide aendern nur die Protokollierung, keinen Hyperparameter.
- hardware/gamepad.py: der Tastatur-Fallback hat nie funktioniert, weil pygame
  ohne display.set_mode() keine Tastendruecke liefert. Liest jetzt primaer das
  PyBullet-Fenster, sonst oeffnet es ein eigenes. Belegung in REAL_EVAL.md.
- Messdaten und hd-Meshes aus Laborsession 1 (25.08.), ar10.py-Indexfix,
  Input-Neukalibrierung.

Co-Authored-By: Claude Opus 5 <noreply@anthropic.com>

File: assets/ar10_description/urdf/ar10.urdf (robot description, URDF)
Before this commit: robot ar10, 35 links, 34 joints
Links:
- link finger1.1a: geometry collision mesh filename=package://ar10_description/meshes/hd/45mm_3_hole/piece_00.o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 scale=0.001 0.001 0.001; collision mesh filename=package://ar10_description/meshes/hd/45mm_3_hole/piece_00.o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 scale=0.001 0.001 0.001
- link finger1.1b: geometry collision mesh filename=package://ar10_description/meshes/hd/30mmROSFULL/piece_00.o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 scale=0.001 0.001 0.001; collision mesh filename=package://ar10_description/meshes/hd/30mmROSFULL/piece_00.o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 scale=0.001 0.001 0.001
- link finger1.1c: geometry collision mesh filename=package://ar10_description/meshes/hd/Fingertip/piece_00.obj scale=0.001 0.001 0.001; collision mesh filename=package://ar10_description/meshes/hd/Fingertip/piece_00.obj scale=0.001 0.001 0.001
- link finger2.1a: geometry collision mesh filename=package://ar10_description/meshes/hd/45mm_3_hole/piece_00.o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 scale=0.001 0.001 0.001; collision mesh filename=package://ar10_description/meshes/hd/45mm_3_hole/piece_00.o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 scale=0.001 0.001 0.001
- link finger2.1b: geometry collision mesh filename=package://ar10_description/meshes/hd/30mmROSFULL/piece_00.o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 scale=0.001 0.001 0.001; collision mesh filename=package://ar10_description/meshes/hd/30mmROSFULL/piece_00.o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 scale=0.001 0.001 0.001
- link finger2.1c: geometry collision mesh filename=package://ar10_description/meshes/hd/Fingertip/piece_00.obj scale=0.001 0.001 0.001; collision mesh filename=package://ar10_description/meshes/hd/Fingertip/piece_00.obj scale=0.001 0.001 0.001
- link finger3.1a: geometry collision mesh filename=package://ar10_description/meshes/hd/45mm_3_hole/piece_00.o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 scale=0.001 0.001 0.001; collision mesh filename=package://ar10_description/meshes/hd/45mm_3_hole/piece_00.o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 scale=0.001 0.001 0.001
- link finger3.1b: geometry collision mesh filename=package://ar10_description/meshes/hd/30mmROSFULL/piece_00.o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 scale=0.001 0.001 0.001; collision mesh filename=package://ar10_description/meshes/hd/30mmROSFULL/piece_00.o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 scale=0.001 0.001 0.001
- link finger3.1c: geometry collision mesh filename=package://ar10_description/meshes/hd/Fingertip/piece_00.obj scale=0.001 0.001 0.001; collision mesh filename=package://ar10_description/meshes/hd/Fingertip/piece_00.obj scale=0.001 0.001 0.001
- link finger4.1a: geometry collision mesh filename=package://ar10_description/meshes/hd/45mm_3_hole/piece_00.o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 scale=0.001 0.001 0.001; collision mesh filename=package://ar10_description/meshes/hd/45mm_3_hole/piece_00.o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 scale=0.001 0.001 0.001
- link finger4.1b: geometry collision mesh filename=package://ar10_description/meshes/hd/30mmROSFULL/piece_00.o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 scale=0.001 0.001 0.001; collision mesh filename=package://ar10_description/meshes/hd/30mmROSFULL/piece_00.o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 scale=0.001 0.001 0.001
- link finger4.1c: geometry collision mesh filename=package://ar10_description/meshes/hd/Fingertip/piece_00.obj scale=0.001 0.001 0.001; collision mesh filename=package://ar10_description/meshes/hd/Fingertip/piece_00.obj scale=0.001 0.001 0.001
- link fingertip1: geometry collision mesh filename=package://ar10_description/meshes/hd/fingertip_v9/piece_00.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 scale=0.001 0.001 0.001; visual mesh filename=package://ar10_description/meshes/fingertip-v9.STL scale=.001 .001 .001
- link fingertip2: geometry collision mesh filename=package://ar10_description/meshes/hd/fingertip_v9/piece_00.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 scale=0.001 0.001 0.001; visual mesh filename=package://ar10_description/meshes/fingertip-v9.STL scale=.001 .001 .001
- link fingertip3: geometry collision mesh filename=package://ar10_description/meshes/hd/fingertip_v9/piece_00.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 scale=0.001 0.001 0.001; visual mesh filename=package://ar10_description/meshes/fingertip-v9.STL scale=.001 .001 .001
- link fingertip4: geometry collision mesh filename=package://ar10_description/meshes/hd/fingertip_v9/piece_00.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 scale=0.001 0.001 0.001; visual mesh filename=package://ar10_description/meshes/fingertip-v9.STL scale=.001 .001 .001
- link palm: geometry collision mesh filename=package://ar10_description/meshes/hd/Palm_RIGHT/piece_00.obj scale=0.001 0.001 0.001; collision mesh filename=package://ar10_description/meshes/hd/Palm_RIGHT/piece_01.obj scale=0.001 0.001 0.001
- link thumb1: geometry collision mesh filename=package://ar10_description/meshes/hd/Thumb_1/piece_00.obj scale=0.001 0.001 0.001; visual mesh filename=package://ar10_description/meshes/Thumb 1.STL scale=.001 .001 .001
- link thumb2: geometry collision mesh filename=package://ar10_description/meshes/hd/Thumb_2/piece_00.obj scale=0.001 0.001 0.001; collision mesh filename=package://ar10_description/meshes/hd/Thumb_2/piece_01.obj scale=0.001 0.001 0.001
- link thumb3.1: geometry collision mesh filename=package://ar10_description/meshes/hd/Thumb_3_Rev2/piece_00.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 scale=0.001 0.001 0.001; collision mesh filename=package://ar10_description/meshes/hd/Thumb_3_Rev2/piece_00.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 scale=0.001 0.001 0.001
- link thumbtip: geometry collision mesh filename=package://ar10_description/meshes/hd/fingertip_v9/piece_00.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 scale=0.001 0.001 0.001; visual mesh filename=package://ar10_description/meshes/fingertip-v9.STL scale=.001 .001 .001

File: assets/benchmark_parts/benchmark_part_1.urdf (robot description, URDF)
Before this commit: robot benchmark_part_1, 1 links, 0 joints
Links:
- link base_link: geometry collision mesh filename=benchmark_parts_stl/hd/part_1/piece_00.obj scale=0.001 0.001 0.001; collision mesh filename=benchmark_parts_stl/hd/part_1/piece_01.obj scale=0.001 0.001 0.001

File: assets/benchmark_parts/benchmark_part_10.urdf (robot description, URDF)
Before this commit: robot benchmark_part_10, 1 links, 0 joints
Links:
- link base_link: geometry collision mesh filename=benchmark_parts_stl/hd/part_10/piece_00.obj scale=0.001 0.001 0.001; collision mesh filename=benchmark_parts_stl/hd/part_10/piece_01.obj scale=0.001 0.001 0.001

File: assets/benchmark_parts/benchmark_part_11.urdf (robot description, URDF)
Before this commit: robot benchmark_part_11, 1 links, 0 joints
Links:
- link base_link: geometry collision mesh filename=benchmark_parts_stl/hd/part_11/piece_00.obj scale=0.001 0.001 0.001; collision mesh filename=benchmark_parts_stl/hd/part_11/piece_01.obj scale=0.001 0.001 0.001

File: assets/benchmark_parts/benchmark_part_12.urdf (robot description, URDF)
Before this commit: robot benchmark_part_12, 1 links, 0 joints
Links:
- link base_link: geometry collision mesh filename=benchmark_parts_stl/hd/part_12/piece_00.obj scale=0.001 0.001 0.001; visual mesh filename=benchmark_parts_stl/benchmark_part_12.stl scale=0.001 0.001 0.001

File: assets/benchmark_parts/benchmark_part_13.urdf (robot description, URDF)
Before this commit: robot benchmark_part_13, 1 links, 0 joints
Links:
- link base_link: geometry collision mesh filename=benchmark_parts_stl/hd/part_13/piece_00.obj scale=0.001 0.001 0.001; collision mesh filename=benchmark_parts_stl/hd/part_13/piece_01.obj scale=0.001 0.001 0.001

File: assets/benchmark_parts/benchmark_part_14.urdf (robot description, URDF)
Before this commit: robot benchmark_part_14, 1 links, 0 joints
Links:
- link base_link: geometry collision mesh filename=benchmark_parts_stl/hd/part_14/piece_00.obj scale=0.001 0.001 0.001; collision mesh filename=benchmark_parts_stl/hd/part_14/piece_01.obj scale=0.001 0.001 0.001

File: assets/benchmark_parts/benchmark_part_2.urdf (robot description, URDF)
Before this commit: robot benchmark_part_2, 1 links, 0 joints
Links:
- link base_link: geometry collision mesh filename=benchmark_parts_stl/hd/part_2/piece_00.obj scale=0.001 0.001 0.001; collision mesh filename=benchmark_parts_stl/hd/part_2/piece_01.obj scale=0.001 0.001 0.001

File: assets/benchmark_parts/benchmark_part_3.urdf (robot description, URDF)
Before this commit: robot benchmark_part_3, 1 links, 0 joints
Links:
- link base_link: geometry collision mesh filename=benchmark_parts_stl/hd/part_3/piece_00.obj scale=0.001 0.001 0.001; collision mesh filename=benchmark_parts_stl/hd/part_3/piece_01.obj scale=0.001 0.001 0.001

File: assets/benchmark_parts/benchmark_part_4.urdf (robot description, URDF)
Before this commit: robot benchmark_part_4, 1 links, 0 joints
Links:
- link base_link: geometry collision mesh filename=benchmark_parts_stl/hd/part_4/piece_00.obj scale=0.001 0.001 0.001; collision mesh filename=benchmark_parts_stl/hd/part_4/piece_01.obj scale=0.001 0.001 0.001

File: assets/benchmark_parts/benchmark_part_5.urdf (robot description, URDF)
Before this commit: robot benchmark_part_5, 1 links, 0 joints
Links:
- link base_link: geometry collision mesh filename=benchmark_parts_stl/hd/part_5/piece_00.obj scale=0.001 0.001 0.001; collision mesh filename=benchmark_parts_stl/hd/part_5/piece_01.obj scale=0.001 0.001 0.001

File: assets/benchmark_parts/benchmark_part_6.urdf (robot description, URDF)
Before this commit: robot benchmark_part_6, 1 links, 0 joints
Links:
- link base_link: geometry collision mesh filename=benchmark_parts_stl/hd/part_6/piece_00.obj scale=0.001 0.001 0.001; collision mesh filename=benchmark_parts_stl/hd/part_6/piece_01.obj scale=0.001 0.001 0.001

File: assets/benchmark_parts/benchmark_part_7.urdf (robot description, URDF)
Before this commit: robot benchmark_part_7, 1 links, 0 joints
Links:
- link base_link: geometry collision mesh filename=benchmark_parts_stl/hd/part_7/piece_00.obj scale=0.001 0.001 0.001; collision mesh filename=benchmark_parts_stl/hd/part_7/piece_01.obj scale=0.001 0.001 0.001

File: assets/benchmark_parts/benchmark_part_8.urdf (robot description, URDF)
Before this commit: robot benchmark_part_8, 1 links, 0 joints
Links:
- link base_link: geometry collision mesh filename=benchmark_parts_stl/hd/part_8/piece_00.obj scale=0.001 0.001 0.001; collision mesh filename=benchmark_parts_stl/hd/part_8/piece_01.obj scale=0.001 0.001 0.001

File: assets/benchmark_parts/benchmark_part_9.urdf (robot description, URDF)
Before this commit: robot benchmark_part_9, 1 links, 0 joints
Links:
- link base_link: geometry collision mesh filename=benchmark_parts_stl/hd/part_9/piece_00.obj scale=0.001 0.001 0.001; visual mesh filename=benchmark_parts_stl/benchmark_part_9.stl scale=0.001 0.001 0.001
